Commit message: attach gripper to arm

File: my_robot_description/urdf/arm.gazebo.xacro (robot description, xacro)
@@ -33,3 +33,6 @@
         </plugin>
     </gazebo>
+    <!-- add gripper relative to hand begin-->
+    <xacro:include filename="gripper.gazebo.xacro" />
+    <!-- add gripper relative to hand end-->
 </robot>

File: my_robot_description/urdf/arm.urdf.xacro (robot description, xacro)
@@ -198,3 +198,6 @@
         <dynamics damping="0.05" friction="0.1"/>
     </joint>
+    <!-- add gripper relative to hand begin-->
+    <xacro:include filename="gripper.xacro" />
+    <!-- add gripper relative to hand end-->
 </robot>

File: my_robot_description/urdf/common_properties.xacro (robot description, xacro)
@@ -9,4 +9,10 @@
     <material name="orange">
         <color rgba="1.0 0.5 0.0 1.0"/>
+    </material>
+    <material name="dark_green">
+        <color rgba="0 0.4 0 1"/>
+    </material>
+    <material name="light_green">
+        <color rgba="0 0.6 0 1"/>
     </material>
     <xacro:macro name="box_inertia" params="m x y z o_xyz o_rpy">
