Commit message: 优化底盘和机械臂连接碰撞,修改机械臂关节初始位置

File: my_robot_description/urdf/arm.urdf.xacro (robot description, xacro)
@@ -27,5 +27,5 @@
         </visual>
         <collision>
-            <origin xyz="0.0 0.0 0.0" rpy="0.0 0.0 0.0"/>
+            <origin xyz="0.0 0.0 ${arm_base_height/2}" rpy="0.0 0.0 0.0"/>
             <geometry>
                 <box size="${arm_base_length} ${arm_base_width} ${arm_base_height}"/>
@@ -154,18 +154,18 @@
     </joint>
     <joint name="joint2" type="revolute">
-        <origin xyz="0.0 0.0 ${shoulder_length}" rpy="0.0 1.0 0.0"/>
+        <origin xyz="0.0 0.0 ${shoulder_length}" rpy="0.0 0.5 0.0"/>
         <parent link="shoulder_link"/>
         <child link="arm_link"/>
         <axis xyz="0.0 1.0 0.0"/>
-        <limit lower="0" upper="2.5" effort="1000.0" velocity="1.0"/>
-        <dynamics damping="100" friction="100"/>
+        <limit lower="-2.5" upper="0.6" effort="1000.0" velocity="1.0"/>
+        <dynamics damping="10" friction="10"/>
     </joint>
     <joint name="joint3" type="revolute">
-        <origin xyz="0.0 0.0 ${arm_length}" rpy="0.0 1.0 0.0"/>
+        <origin xyz="0.0 0.0 ${arm_length}" rpy="0.0 0.0 0.0"/>
         <parent link="arm_link"/>
         <child link="elbow_link"/>
         <axis xyz="0.0 1.0 0.0"/>
-        <limit lower="0" upper="2.5" effort="1000.0" velocity="1.0"/>
-        <dynamics damping="30" friction="30"/>
+        <limit lower="-2.5" upper="0.6" effort="1000.0" velocity="1.0"/>
+        <dynamics damping="10" friction="10"/>
     </joint>
     <joint name="joint4" type="revolute">
@@ -175,5 +175,5 @@
         <axis xyz="0.0 0.0 1"/>
         <limit lower="-3.14" upper="3.14" effort="1000.0" velocity="1.0"/>
-        <dynamics damping="20" friction="20"/>
+        <dynamics damping="10" friction="10"/>
     </joint>
     <joint name="joint5" type="revolute">

Commit message: 更改机械臂模型大小及初始姿态

File: my_robot_description/urdf/arm.urdf.xacro (robot description, xacro)
@@ -1,20 +1,20 @@
 <?xml version="1.0"?>
 <robot xmlns:xacro="http://www.ros.org.wiki/xacro">
-    <xacro:property name="arm_base_length" value="0.4" />
-    <xacro:property name="arm_base_width" value="0.4" />
-    <xacro:property name="arm_base_height" value="0.1" />
-    <xacro:property name="shoulder_length" value="0.5" />
-    <xacro:property name="shoulder_radius" value="0.1" />
-    <xacro:property name="arm_length" value="0.6" />
-    <xacro:property name="arm_radius" value="0.05" />
-    <xacro:property name="elbow_length" value="0.1" />
-    <xacro:property name="elbow_radius" value="0.05" />
-    <xacro:property name="forearm_length" value="0.5" />
-    <xacro:property name="forearm_radius" value="0.05" />
-    <xacro:property name="wrist_length" value="0.1" />
-    <xacro:property name="wrist_width" value="0.1" />
-    <xacro:property name="wrist_height" value="0.05" />
-    <xacro:property name="hand_length" value="0.1" />
-    <xacro:property name="hand_width" value="0.1" />
+    <xacro:property name="arm_base_length" value="0.28" />
+    <xacro:property name="arm_base_width" value="0.28" />
+    <xacro:property name="arm_base_height" value="0.08" />
+    <xacro:property name="shoulder_length" value="0.32" />
+    <xacro:property name="shoulder_radius" value="0.07" />
+    <xacro:property name="arm_length" value="0.36" />
+    <xacro:property name="arm_radius" value="0.04" />
+    <xacro:property name="elbow_length" value="0.08" />
+    <xacro:property name="elbow_radius" value="0.04" />
+    <xacro:property name="forearm_length" value="0.32" />
+    <xacro:property name="forearm_radius" value="0.04" />
+    <xacro:property name="wrist_length" value="0.08" />
+    <xacro:property name="wrist_width" value="0.08" />
+    <xacro:property name="wrist_height" value="0.04" />
+    <xacro:property name="hand_length" value="0.08" />
+    <xacro:property name="hand_width" value="0.08" />
     <xacro:property name="hand_height" value="0.02" />
     <link name="arm_base_link">
@@ -32,5 +32,5 @@
             </geometry>
         </collision>
-        <xacro:box_inertia m="3.0" x="${arm_base_length}" y="${arm_base_width}" z="${arm_base_height}"
+        <xacro:box_inertia m="1.5" x="${arm_base_length}" y="${arm_base_width}" z="${arm_base_height}"
                            o_xyz="0.0 0.0 ${arm_base_height/2.0}" o_rpy="0 0 0" />
     </link>
@@ -49,5 +49,5 @@
             </geometry>
         </collision>
-        <xacro:cylinder_inertia m="1.5" r="${shoulder_radius}" h="${shoulder_length}"
+        <xacro:cylinder_inertia m="0.8" r="${shoulder_radius}" h="${shoulder_length}"
                                 o_xyz="0.0 0.0 ${shoulder_length/2.0}" o_rpy="0 0 0" />
     </link>
@@ -66,5 +66,5 @@
             </geometry>
         </collision>
-        <xacro:cylinder_inertia m="1.0" r="${arm_radius}" h="${arm_length}"
+        <xacro:cylinder_inertia m="0.5" r="${arm_radius}" h="${arm_length}"
                                 o_xyz="0.0 0.0 ${arm_length/2.0}" o_rpy="0 0 0" />
     </link>
@@ -100,5 +100,5 @@
             </geometry>
         </collision>
-        <xacro:cylinder_inertia m="0.5" r="${forearm_radius}" h="${forearm_length}"
+        <xacro:cylinder_inertia m="0.3" r="${forearm_radius}" h="${forearm_length}"
                                 o_xyz="0.0 0.0 ${forearm_length/2.0}" o_rpy="0 0 0" />
     </link>
@@ -140,5 +140,5 @@
     </link>
     <joint name="base_arm_joint" type="fixed">
-        <origin xyz="0.0 0.0 ${base_height}" rpy="0.0 0.0 0.0"/>
+        <origin xyz="${base_length/2 - arm_base_length/1.5} 0.0 ${base_height}" rpy="0.0 0.0 0.0"/>
         <parent link="base_link"/>
         <child link="arm_base_link"/>
@@ -162,9 +162,9 @@
     </joint>
     <joint name="joint3" type="revolute">
-        <origin xyz="0.0 0.0 ${arm_length}" rpy="0.0 0.0 0.0"/>
+        <origin xyz="0.0 0.0 ${arm_length}" rpy="0.0 2.3 0.0"/>
         <parent link="arm_link"/>
         <child link="elbow_link"/>
         <axis xyz="0.0 1.0 0.0"/>
-        <limit lower="-2.5" upper="0.6" effort="1000.0" velocity="1.0"/>
+        <limit lower="-2.5" upper="2.5" effort="1000.0" velocity="1.0"/>
         <dynamics damping="10" friction="10"/>
     </joint>

Commit message: 更新机器人模型，确保camera opencv 识别和lidar 扫描都正常

File: my_robot_description/urdf/arm.urdf.xacro (robot description, xacro)
@@ -3,5 +3,5 @@
     <xacro:property name="arm_base_length" value="0.28" />
     <xacro:property name="arm_base_width" value="0.28" />
-    <xacro:property name="arm_base_height" value="0.08" />
+    <xacro:property name="arm_base_height" value="0.12" />
     <xacro:property name="shoulder_length" value="0.32" />
     <xacro:property name="shoulder_radius" value="0.07" />

File: my_robot_description/urdf/camera.xacro (robot description, xacro)
@@ -29,5 +29,5 @@
         <parent link="base_link"/>
         <child link="camera_link"/>
-        <origin xyz="${(base_length + camera_length)/2.0} 0 ${base_height/3.0}" rpy="0.0 0.0 0.0"/>
+        <origin xyz="${(base_length + camera_length)/2.0} 0 ${base_height/2.0}" rpy="0.0 0.0 0.0"/>
     </joint>
     <gazebo reference="camera_link">
