Commit message: 夹爪右指无法滑动问题修复,夹爪相关状态修改

File: my_robot_description/urdf/gripper.gazebo.xacro (robot description, xacro)
@@ -4,10 +4,101 @@
         <material>Gazebo/DarkGreen</material>
     </gazebo>
+    <!-- 指面接触参数。
+         注意别把 kp / mu 调得太硬太高：gz_ros2_control 的位置指令内部是速度量
+         （v = position_proportional_gain × 误差，默认增益 0.1），指爪移动很慢，
+         接触过硬 + 摩擦过高会让指爪被静摩擦"锁死"（详见 gripper.xacro 里
+         关于指爪关节 z 间隙的说明）。这里的值故意与方块自身(mu=0.8)同量级。
+         仿真里真正可靠的抓取靠 DetachableJoint 吸附（见 PICK_PLACE.md），
+         摩擦抓取只是备选路径。 -->
     <gazebo reference="gripper_left_finger_link">
         <material>Gazebo/LightGreen</material>
+        <mu1>0.8</mu1>
+        <mu2>0.8</mu2>
+        <kp>100000.0</kp>
+        <kd>10.0</kd>
     </gazebo>
     <gazebo reference="gripper_right_finger_link">
         <material>Gazebo/LightGreen</material>
+        <mu1>0.8</mu1>
+        <mu2>0.8</mu2>
+        <kp>100000.0</kp>
+        <kd>10.0</kd>
     </gazebo>
     <!-- 夹爪关节状态已由 gz_ros2_control 经 joint_state_broadcaster 提供，不再使用 GZ JointStatePublisher -->
+    <!-- ============================================================
+         仿真专用补丁：用 Gazebo 自带的 JointPositionController 直接驱动右指
+         ============================================================
+         现象：本仿真后端（Ignition Gazebo 6 / Fortress）下，名叫
+         gripper_right_finger_joint 的关节经 gz_ros2_control 完全驱动不了 ——
+         接口 available/claimed、控制器里也含它、JTC 的 error 显示确实在命令它，
+         但关节状态恒为 0（连数值噪声都没有），指爪物理上不动；
+         而 gripper_left_finger_joint 一切正常。
+         根因（已用干净的隔离实验定论）：决定因素是**关节的「轴方向 + 限位取向」组合**
+         —— 只有与左指完全同构的形态（轴 +1、限位 [0, +X]、正向命令）能被驱动：
+           axis +1 + limits [0, 0.06]  → 能动（左指）
+           axis +1 + limits [-0.06, 0] → 不动（右指的原始设计就是这种！）
+           axis -1 + limits [0, 0.06]  → 不动
+         已排除（独立 ROS_DOMAIN_ID + 先摘掉 mirror 后复现）：关节名、<ros2_control>
+         声明顺序、URDF 关节定义顺序、关节 origin、接触摩擦参数、控制器里放几个关节、
+         MoveIt。右指要向内合拢就必须用负向轴或负限位，而这两种恰好都驱动不了，
+         所以仿真里需要下面这条镜像通路。
+         （修正记录：早先写成「按名字绑错实体」是过度推断 —— 交换 origin 时轴是跟着
+         关节名一起走的，我把「轴 −1 不动」误读成了「名字叫 right 的不动」。）
+         这里给右指挂一个 Gazebo 原生插件，它自己按名字在本模型里找关节并
+         直接写位置，是一条独立于 gz_ros2_control 的通路；
+         再由 my_robot_bringup 的 gripper_mirror 节点把左指位置镜像到
+         /gripper_right_finger_cmd，两个指爪就能同步开合。
+         本插件 + mirror 是可用的绕过方案（已实测两指跟随误差 ≤0.6mm）。
+         注意：这只影响仿真。真机上两个指关节都由 ros2_control 正常驱动，
+         ros2_control 侧的配置（双指都在 gripper_controller 里）保持不变。
+         一旦 gz_ros2_control 修好这个问题，删掉本插件 + 桥接 + mirror 节点即可。
+         ============================================================ -->
+    <gazebo>
+        <plugin filename="ignition-gazebo-joint-position-controller-system"
+                name="ignition::gazebo::systems::JointPositionController">
+            <joint_name>gripper_right_finger_joint</joint_name>
+            <topic>/gripper_right_finger_cmd</topic>
+            <initial_position>0.0</initial_position>
+            <p_gain>400</p_gain>
+            <i_gain>8</i_gain>
+            <d_gain>40</d_gain>
+            <i_max>5.0</i_max>
+            <i_min>-5.0</i_min>
+            <cmd_max>100.0</cmd_max>
+            <cmd_min>-100.0</cmd_min>
+        </plugin>
+    </gazebo>
+    <!-- ============================================================
+         可选：DetachableJoint 吸附（仿真里保证抓取可靠）
+         ============================================================
+         Gazebo 里的摩擦抓取成功率有限（指爪打滑、方块被顶飞、接触穿透），
+         所以抓取时把方块和夹爪之间硬连一个 fixed joint，松爪时再断开。
+         视觉/规划/状态机代码完全不用改，只在夹紧/松开那一刻多发一条消息。
+         用 xacro 参数 use_detachable 控制是否包含本插件（默认关，
+         由 my_robot_gazebo.launch.xml 的 use_detachable 参数传进来），
+         因为插件在 Configure 时就会把两者连起来，需要 orchestrator 上电后
+         先发一次 detach 抵消（见 my_robot_task_orchestrator/orchestrator.py）。
+         attach/detach 话题是 Gazebo 传输层话题，经 gazebo_bridge.yaml
+         桥接成 ROS 的 std_msgs/Empty。
+         ============================================================ -->
+    <xacro:if value="$(arg use_detachable)">
+        <gazebo>
+            <plugin filename="ignition-gazebo-detachable-joint-system"
+                    name="ignition::gazebo::systems::DetachableJoint">
+                <!-- 注意这里必须写 hand_link，不能写 gripper_base_link：
+                     URDF→SDF 转换会把固定关节合并（lump），gripper_base_link 被
+                     并进 hand_link，运行时模型里根本没有 gripper_base_link 这个名字，
+                     插件会报 "Link with name gripper_base_link not found ...
+                     Failed to initialize"。hand_link 携带了合并后的夹爪底板碰撞体，
+                     几何上就是夹爪本体，等价。 -->
+                <parent_link>hand_link</parent_link>
+                <child_model>red_cube</child_model>
+                <child_link>red_cube_link</child_link>
+                <attach_topic>/red_cube/attach</attach_topic>
+                <detach_topic>/red_cube/detach</detach_topic>
+                <output_topic>/red_cube/detachable_joint_state</output_topic>
+                <suppress_child_warning>true</suppress_child_warning>
+            </plugin>
+        </gazebo>
+    </xacro:if>
 </robot>

File: my_robot_description/urdf/gripper.xacro (robot description, xacro)
@@ -57,4 +57,13 @@
         <origin xyz="0 0 0" rpy="0 0 0"/>
     </joint>
+    <!-- 指爪关节 origin 的 z = 0.02（原始设计，保持不动）。
+         曾经一度改成 0.03 想"消除指爪与夹爪底板的零间隙接触"，**那是错的**：
+         后续实验证明右指不动与接触参数无关（详见下面 gripper_right_finger_joint
+         的说明），真正原因是 mimic 被丢弃 + gz_ros2_control 对该关节名的写通路缺陷。
+         实测把 z 改回 0.02 之后夹爪开合依然完全正常。
+         注意这个 z 会决定抓取时工具该降到多高（见 PICK_PLACE.md 第六节）：
+         指爪碰撞体在 gripper/tool 系里占 z ∈ [0.02, 0.10]（关节 z + 连杆内偏移
+         0.04 ± 0.04），工具 +Z 朝下时指爪底端落在世界 z = tool_z - 0.10，
+         所以台面 0.40 上抓方块时 tool_z = 0.50 刚好贴到台面且完整包住方块。 -->
     <joint name="gripper_left_finger_joint" type="prismatic">
         <parent link="gripper_base_link"/>
@@ -68,7 +77,24 @@
         <child link="gripper_right_finger_link"/>
         <origin xyz="0.07 0 0.02" rpy="0 0 0"/>
-        <axis xyz="1 0 0"/>
-        <limit lower="-0.06" upper="0.0" effort="1000" velocity="1.0"/>
-        <mimic joint="gripper_left_finger_joint" multiplier="-1"/>
+        <!-- 轴取 -X：正值 = 指爪朝中心合拢。这样两个指关节的约定完全一致
+             （限位都是 [0, 0.06]、正值都是合拢），上层/ SRDF 里两个关节
+             给相同的正值即可，不用再记一个取负、一个取正。
+             原来这里是 axis="1 0 0" + limit [-0.06, 0]（正值=张开），
+             实测在 Ignition Gazebo 6 下该关节的命令完全不被执行
+             （左指正常跟随，右指恒定停在 0），改成与左指同构后正常。 -->
+        <axis xyz="-1 0 0"/>
+        <limit lower="0" upper="0.06" effort="1000" velocity="1.0"/>
+        <!-- 这里原本是 <mimic joint="gripper_left_finger_joint" multiplier="-1"/>，
+             已移除。原因：本仿真后端是 Ignition Gazebo 6 (Fortress)，其
+             sdformat12 的 SDF 1.9 规范里没有 mimic 元素，URDF 经
+             `ros_gz_sim create -topic robot_description` 转 SDF 时 mimic 会被丢弃，
+             右指变成无驱动、无约束的自由关节 —— 合爪时只有左指动、右指被推着乱跑，
+             夹不住任何东西。
+             现在改为双指都由 gripper_controller 直接驱动（见
+             my_robot.ros2_control.xacro）：
+               合到 5cm 方块 → 两指都 +0.035
+               完全闭合     → 两指都 +0.060
+             对应 SRDF 的 gripper_grasp / gripper_closed 命名目标。
+             注意：不要把 mimic 加回来，除非换到支持它的仿真后端。 -->
     </joint>
 </robot>

File: my_robot_description/urdf/my_robot.ros2_control.xacro (robot description, xacro)
@@ -49,4 +49,17 @@
             </state_interface>
         </joint>
+        <!-- 右指也必须纳入 ros2_control：
+             gripper.xacro 里右指原本用 URDF <mimic joint="gripper_left_finger_joint">
+             跟随左指，但本仿真后端 Ignition Gazebo 6 (Fortress) / sdformat12
+             的 SDF 1.9 规范里没有 mimic 元素，URDF 转 SDF 时 mimic 被丢弃，
+             右指成了一个没有驱动、没有约束的自由滑动关节 —— 表现为"合爪时
+             只有左指动、右指被推着乱跑、夹不住物体"。这里改成双指都直接驱动，
+             由 gripper_controller 同时给两个关节发位置指令。 -->
+        <joint name="gripper_right_finger_joint">
+            <command_interface name="position"/>
+            <state_interface name="position">
+                <param name="initial_value">0.0</param>
+            </state_interface>
+        </joint>
     </ros2_control>
     <!-- 注意：MobileBase（差速轮）不纳入 ros2_control，

File: my_robot_moveit_config/config/my_robot.ros2_control.xacro (robot description, xacro)
@@ -50,4 +50,10 @@
                 </state_interface>
             </joint>
+            <joint name="gripper_right_finger_joint">
+                <command_interface name="position"/>
+                <state_interface name="position">
+                  <param name="initial_value">${initial_positions['gripper_right_finger_joint']}</param>
+                </state_interface>
+            </joint>
         </ros2_control>
     </xacro:macro>
