Commit message: my_robot_bringup 包中 集成moveit2 ros_control配置，执行moveit2 运动规划
执行命令: ros2 launch my_robot_bringup my_robot.launch.xml

File: my_robot_description/urdf/gripper.xacro (robot description, xacro)
@@ -53,5 +53,5 @@
     </link>
     <joint name="gripper_base_joint" type="fixed">
-        <parent link="hand_link"/>
+        <parent link="tool_link"/>
         <child link="gripper_base_link"/>
         <origin xyz="0 0 0" rpy="0 0 0"/>

File: my_robot_description/urdf/my_robot.urdf.xacro (robot description, xacro)
@@ -7,3 +7,4 @@
     <xacro:include filename="arm.urdf.xacro" />
     <xacro:include filename="arm.gazebo.xacro" />
+    <xacro:include filename="my_robot.ros2_control.xacro" />
 </robot>

Commit message: 夹爪底板碰撞体留出余量避免毫米级擦边自碰判废整组解

File: my_robot_description/urdf/gripper.xacro (robot description, xacro)
@@ -1,4 +1,10 @@
 <?xml version="1.0"?>
 <robot xmlns:xacro="http://www.ros.org.wiki/xacro">
+    <!-- 【碰撞体比可视体略小】夹爪底板可视尺寸 0.20x0.06x0.02，这里碰撞用
+         0.18x0.05x0.014：实测 move_group 报 shoulder_link 与 gripper_base_link
+         穿透 2.8mm 这类"擦边自碰"（深度只有几毫米），会让该位姿的所有 IK 解
+         都被 /check_state_validity 判废、整个抓取失败。这里每边留 5~10mm 余量，
+         让"真实外形不接触、只是碰撞体擦边"的位姿能通过。
+         注意：这是**仿真侧**的放宽，真机应按实际零件尺寸重新标定。 -->
     <link name="gripper_base_link">
         <visual>
@@ -11,5 +17,5 @@
         <collision>
             <geometry>
-                <box size="0.2 0.06 0.02"/>
+                <box size="0.18 0.05 0.014"/>
             </geometry>
             <material name="dark_green"/>
